File: learner-pcb.kicad_pcb (KiCad board)
At the start: 2 copper layers, 1 part, among them U1 ATmega32U4-AU

Commit message: finish first pass at pcb.
Parts:
- added C1: 22pF, Capacitor_SMD:C_0805_2012Metric, B.Cu at (265.2, -174.1)
- added C2: 22pF, Capacitor_SMD:C_0805_2012Metric, B.Cu at (254.9, -174.2)
- added C3: 1uF, Capacitor_SMD:C_0805_2012Metric, B.Cu at (249.3, -162.3)
- added C4: 0.1uF, Capacitor_SMD:C_0805_2012Metric, B.Cu at (252.2, -170.1)
- added C5: 0.1uF, Capacitor_SMD:C_0805_2012Metric, B.Cu at (268.4, -166.4)
- added C6: 0.1uF, Capacitor_SMD:C_0805_2012Metric, B.Cu at (263.8, -153.4)
- added C7: 10uF, Capacitor_SMD:C_0805_2012Metric, B.Cu at (255.3, -153.2)
- added D1: SOD-123, Diode_SMD:D_SOD-123, B.Cu at (288.2, -172.6)
- added D2: SOD-123, Diode_SMD:D_SOD-123, B.Cu at (307.2, -172.6)
- added D3: SOD-123, Diode_SMD:D_SOD-123, B.Cu at (288.2, -153.6)
- added D4: SOD-123, Diode_SMD:D_SOD-123, B.Cu at (307.2, -153.6)
- added F1: 500mA, Fuse:Fuse_1206_3216Metric, B.Cu at (234.4, -164.9)
- added MX1: MX-NoLED, MX_Alps_Hybrid:MX-1U, F.Cu at (280.3, -172.6)
- added MX2: MX-NoLED, MX_Alps_Hybrid:MX-1U, F.Cu at (299.3, -172.6)
- added MX3: MX-NoLED, MX_Alps_Hybrid:MX-1U, F.Cu at (280.2, -153.7)
- added MX4: MX-NoLED, MX_Alps_Hybrid:MX-1U, F.Cu at (299.2, -153.7)
- added R1: 10k, Resistor_SMD:R_0805_2012Metric, B.Cu at (249.4, -170.1)
- added R2: 22, Resistor_SMD:R_0805_2012Metric, B.Cu at (241.8, -168.5)
- added R3: 22, Resistor_SMD:R_0805_2012Metric, B.Cu at (238.5, -168.5)
- added R4: 10k, Resistor_SMD:R_0805_2012Metric, B.Cu at (268.4, -156.8)
- added SW1: SW_Push, random-keyboard-parts:SKQG-1155865, B.Cu at (237.5, -148.6)
- added USB1: Molex-0548190589, random-keyboard-parts:Molex-0548190589, B.Cu at (240.7, -180.8)
- added Y1: 16MHz, Crystal:Crystal_SMD_3225-4Pin_3.2x2.5mm, B.Cu at (260.0, -174.2)
- U1: moved to B.Cu
- moved U1 83.2 mm to (259.7, -161.5)
Connections:
- U1 pad 27: Net-(U1-Pad27) -> COL0
- U1 pad 28: Net-(U1-Pad28) -> ROW0
- U1 pad 29: Net-(U1-Pad29) -> COL1
- U1 pad 30: Net-(U1-Pad30) -> ROW1
Routing:
- net GND: track 0.00 -> 127.7 mm, vias 0 -> 2
- net +5V: track 0.00 -> 87.1 mm, vias 0 -> 6
- net COL1: track 0.00 -> 50.8 mm
- net ROW1: track 0.00 -> 50.0 mm
- net ROW0: track 0.00 -> 46.2 mm
- net Net-(R1-Pad2): track 0.00 -> 42.0 mm, vias 0 -> 3
- net COL0: track 0.00 -> 36.6 mm
- net Net-(R3-Pad1): track 0.00 -> 20.1 mm
- net Net-(R2-Pad1): track 0.00 -> 19.0 mm
- net VCC: track 0.00 -> 17.2 mm
- net Net-(C2-Pad1): track 0.00 -> 12.7 mm
- net Net-(C1-Pad1): track 0.00 -> 10.8 mm
- net D-: track 0.00 -> 7.18 mm
- net D+: track 0.00 -> 7.06 mm
- net Net-(D3-Pad2): track 0.00 -> 6.60 mm
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Other:
- board outline added: 76.8 x 38.4 mm
- net class Default: trace_width 0.25 -> 0.254
- net class Power added: clearance 0.2, trace_width 0.381, via_dia 0.8, via_drill 0.4
